File: flacplayer.kicad_sch (KiCad schematic)
At the start: 16 parts, among them IC1 CS43131-CNZR, J1 AudioJack3, J2 USB_C_Receptacle_USB2.0, Q1 Q_Dual_NMOS_G1S2G2D2S1D1, U1 ESP32-S3-MINI-1, U2 MAX17048X, U3 AMS1117-3.3, U4 DW01A

Commit message: journals and some other stuffH
Parts:
- removed IC1: CS43131-CNZR, QFN40P500X500X80-41N, symbol CS43131-CNZR:CS43131-CNZR
- added C10: 100nF, symbol Device:C_Small
- added C11, C12, C13, C5, C7, C9: 1uF, symbol Device:C_Small
- added C14, C15: 2.2uF, symbol Device:C_Small
- added C16, C17: 4.7uF, symbol Device:C_Small
- added C4: 0.1uF, symbol Device:C_Small
- added C6, C8: 10uF, symbol Device:C_Small
- added D1, D2: D_Small, symbol Device:D_Small
- added R5: 4.7k, symbol Device:R_Small
- added R6: 2k, symbol Device:R_Small
- added U5: TAD5242, Library:Texas_RGE0024R_VQFN-24-1EP_4x4mm_P0.5mm_EP2.1x2.1mm, symbol TAD5242:TAD5242
- added U6: TPA6132A2RTE, Package_DFN_QFN:WQFN-16-1EP_3x3mm_P0.5mm_EP1.6x1.6mm_ThermalVias, symbol Amplifier_Audio:TPA6132A2RTE
- added U7: MCP73831-2-OT, Package_TO_SOT_SMD:SOT-23-5, symbol Battery_Management:MCP73831-2-OT
Connections:
- net +3V3: now also C15.2, C5.1, C6.1, U5.6 (IOVDD), U5.7 (MD1), U5.8 (MD2), U6.14 (VDD)
- net +BATT: now also U2.2 (CELL), U2.3 (VDD), C16.1, C4.1, D2.2 (A), U7.3 (V_{BAT})
- net D+: now also U1.24 (USB_D+)
- net D-: now also U1.23 (USB_D-)
- net GND: now also J1.S, U1.1 (GND), U1.2 (GND), U1.42 (GND), U1.43 (GND), U1.46 (GND), U1.47 (GND), U1.48 (GND), U1.49 (GND), U1.50 (GND), U1.51 (GND), U1.52 (GND), U1.53 (GND), U1.54 (GND), U1.55 (GND), U1.56 (GND), U1.57 (GND), U1.58 (GND), U1.59 (GND), U1.60 (GND), U1.61 (GND), U1.62 (GND), U1.63 (GND), U1.64 (GND), U1.65 (GND), U2.1 (CTG), U2.4 (GND), U2.6 (QSTRT), C10.2, C11.2, C12.2, C14.1, C15.1, C16.2, C17.2, C4.2, C5.2, C6.2, C7.2, C8.2, C9.2, R5.1, R6.2, U5.10 (MD4), U5.12 (MD5), U5.14 (VSSA), U5.15 (VSSA), U5.16 (VSSA), U5.17 (VSSA), U5.18 (VSSA), U5.25 (VSS), U5.4 (MD6), U5.9 (MD3), U5.A1 (VSS), U5.A2 (VSS), U5.A3 (VSS), U5.A4 (VSS), U6.10 (PGND), U6.15 (SGND), U6.17 (EP), U7.2 (V_{SS})
- net VBUS: now also C17.1, D1.2 (A), U7.4 (V_{DD}); no longer C2.1, U3.3 (VI)
- net RIGHT: now reaches J1.R
- net RIGHT: now also U6.5 (OUTR)
- net LEFT: now reaches J1.T
- net LEFT: now also U6.16 (OUTL)
- net FSYNC: now reaches U1.28 (IO33)
- net FSYNC: now also U5.3 (FSYNC)
- net BCLK: now reaches U1.29 (IO34)
- net BCLK: now also U5.2 (BCLK)
- net DIN: now reaches U1.31 (IO35)
- net DIN: now also U5.5 (DIN)
- net ~{ARLT}: now reaches U2.5 (~{ALRT})
- net SCL: now reaches U2.7 (SCL)
- net SDA: now reaches U2.8 (SDA)
- new net: R6.1, U7.5 (PROG)
- new net: C10.1, C11.1, U5.1 (DREG)
- new net: C2.1, D1.1 (K), D2.1 (K), U3.3 (VI)
- new net: R5.2, U5.13 (MD0)
- new net: C9.1, U5.24 (VREF)
- new net: C13.1, U6.11 (CPP)
- new net: C14.2, U6.12 (HPVDD)
- new net: C12.1, U6.8 (HPVSS)
- new net: C13.2, U6.9 (CPN)
- new net +3.3VA: C7.1, C8.1, U5.23 (AVDD)
- new net OUTA+: U5.20 (OUT1+), U6.3 (INR+)
- new net OUTA-: U5.19 (OUT1-), U6.4 (INR-)
- new net OUTB+: U5.21 (OUT2+), U6.2 (INL+)
- new net OUTB-: U5.22 (OUT2-), U6.1 (INL-)
- no-connect marks 2 -> 4
Other:
- note added: "Audio"
- moved on the sheet: BT1, C1, C2, C3, J1, J2, Q1A, Q1B, R1, R2, R3, R4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

Commit message: meow mrow :3
Parts:
- added C18, C19, C20, C21, C22, C23, C24, C25, C26, C27, C28, C29: 1uF, symbol Device:C_Small
- added C30, C31: 4.7uF, symbol Device:C_Small
- added D3, D4, D5: D_Schottky, symbol Device:D_Schottky_Small
- added J3: Conn_01x25, symbol Connector_Generic:Conn_01x25
- added L1: 68uH, symbol Device:L_Small
- added Q2: IRLML2060, Package_TO_SOT_SMD:SOT-23, symbol Transistor_FET:IRLML2060
- added R7: 0.47r, symbol Device:R_Small
- added R8: 10k, symbol Device:R_Small
Connections:
- net +3V3: now also U1.3 (3V3), C20.1, C30.1, J3.15 (Pin_15), J3.16 (Pin_16), L1.1
- net DIN: now also J3.14 (Pin_14)
- net GND: now also C18.2, C19.2, C20.2, C21.2, C22.2, C23.2, C24.2, C25.2, C26.2, C27.2, C28.2, C29.2, C30.2, D5.1 (K), J3.8 (Pin_8), R7.2, R8.1
- net SCL: now also U1.33 (IO37)
- net SDA: now also U1.32 (IO36)
- net ~{ARLT}: now also U1.34 (IO38)
- new net: C31.1, D3.2 (A), L1.2, Q2.2 (S)
- new net: C24.1, J3.20 (Pin_20)
- new net: C21.1, J3.17 (Pin_17)
- new net: C22.1, J3.18 (Pin_18)
- new net: C26.1, J3.22 (Pin_22)
- new net: C19.1, J3.5 (Pin_5)
- new net: C23.1, J3.19 (Pin_19)
- new net: C27.1, J3.23 (Pin_23)
- new net: C29.1, J3.25 (Pin_25)
- new net: C18.1, J3.4 (Pin_4)
- new net: C31.2, D4.1 (K), D5.2 (A)
- new net BUSY: J3.9 (Pin_9)
- new net CLK: J3.13 (Pin_13)
- new net CS: J3.12 (Pin_12)
- new net DC: J3.11 (Pin_11)
- new net GDR: J3.2 (Pin_2), Q2.1 (G), R8.2
- new net PREVGH: C25.1, D3.1 (K), J3.21 (Pin_21)
- new net PREVGL: C28.1, D4.2 (A), J3.24 (Pin_24)
- new net RESE: J3.3 (Pin_3), Q2.3 (D), R7.1
- new net RST: J3.10 (Pin_10)
- no-connect marks 4 -> 7
Other:
- moved on the sheet: BT1, C1, C16, C17, C2, C3, C4, D1, D2, J2, Q1A, Q1B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

Commit message: does ts work
Parts:
- removed C29: 1uF, symbol Device:C_Small
- removed C3: 0.1uF, symbol Device:C_Small
- removed C30, C31: 4.7uF, symbol Device:C_Small
- removed D3, D4, D5: D_Schottky, symbol Device:D_Schottky_Small
- removed J3: Conn_01x25, symbol Connector_Generic:Conn_01x25
- removed Q1: Q_Dual_NMOS_G1S2G2D2S1D1, symbol Transistor_FET:Q_Dual_NMOS_G1S2G2D2S1D1
- removed Q2: IRLML2060, Package_TO_SOT_SMD:SOT-23, symbol Transistor_FET:IRLML2060
- removed R3: 100, symbol Device:R_Small
- removed R4: 1k, symbol Device:R_Small
- removed U4: DW01A, Package_TO_SOT_SMD:SOT-23-6, symbol Battery_Management:DW01A
- added D3, D4, D5: MBR0530, Diode_SMD:D_SOD-123, symbol Diode:MBR0530
- added J4: Conn_01x24_MountingPin, symbol Connector_Generic_MountingPin:Conn_01x24_MountingPin
- added Q2: AO3400A, Package_TO_SOT_SMD:SOT-23, symbol Transistor_FET:AO3400A
- added R9: 10k, symbol Device:R_Small
- added SW1, SW2, SW3, SW4, SW5, SW6, SW7: SW_Push, symbol Switch:SW_Push
- C18, C21, C22, C23, C24, C26, C27: value 1uF -> 4.7uF/25V
- C19, C20, C25, C28: value 1uF -> 1uF/50V
- C2: value 47uF -> 10uF
- L1: value 68uH -> 10uH
- R7: value 0.47r -> 1Mo
- R8: value 10k -> 2.2o
Connections:
- net PREVGH is gone; now on net GND: C25.1
- net PREVGL is gone; now on net GND: C28.1
- net +3V3: now also C26.2, L1.2, R9.2; no longer C20.1, L1.1
- net BCLK: now also U1.37 (IO41)
- net DIN: now also U1.38 (IO42)
- net FSYNC: now also U1.36 (IO40)
- net GDR: now also J4.2 (Pin_2); no longer R8.2
- net GND: now also C18.1, C19.1, C20.1, C21.1, C22.1, C23.1, C24.1, C26.1, R8.2, D5.1 (K), J4.17 (Pin_17), J4.8 (Pin_8), J4.MP (MountPin), SW1.2, SW2.2, SW3.2, SW4.2, SW5.2, SW6.2, SW7.2; no longer C18.2, C19.2, C20.2, C21.2, C22.2, C23.2, C24.2, C25.2, C26.2, C27.2, C28.2, R8.1
- net RESE: now also R8.1, J4.3 (Pin_3), Q2.2 (S); no longer R7.1
- net EN: now reaches U6.13 (EN)
- net G0: now reaches U6.6 (G0)
- net G1: now reaches U6.7 (G1)
- net at C27.1: now also L1.1, D3.2 (A), Q2.3 (D)
- net EPD_BUSY: now reaches U1.10 (IO6)
- net EPD_BUSY: now also J4.9 (Pin_9)
- net EPD_CS: now reaches U1.14 (IO10)
- net EPD_CS: now also J4.12 (Pin_12)
- net EPD_DIN: now reaches U1.15 (IO11)
- net EPD_DIN: now also J4.14 (Pin_14)
- net EPD_SCK: now reaches U1.16 (IO12)
- net EPD_SCK: now also J4.13 (Pin_13)
- net SW_1: now reaches U1.17 (IO13)
- net SW_1: now also SW1.1
- net SW_VOL+: now reaches U1.18 (IO14)
- net SW_VOL+: now also SW3.1
- net SW_VOL-: now reaches U1.19 (IO15)
- net SW_VOL-: now also SW5.1
- net SW_PP: now reaches U1.20 (IO16)
- net SW_PP: now also SW2.1
- net SW_MENU: now reaches U1.21 (IO17)
- net SW_MENU: now also SW4.1
- net SW_BACK: now reaches U1.22 (IO18)
- net SW_BACK: now also SW6.1
- net ~{RESET}: now reaches U1.45 (EN)
- net ~{RESET}: now also C28.2, R9.1, SW7.1
- net EPD_DC: now reaches U1.8 (IO4)
- net EPD_DC: now also J4.11 (Pin_11)
- net EPD_RST: now reaches U1.9 (IO5)
- net EPD_RST: now also J4.10 (Pin_10)
- net OUTA+: no longer names the net of U5.20 (OUT1+), U6.3 (INR+)
- net OUTA-: no longer names the net of U5.19 (OUT1-), U6.4 (INR-)
- net OUTB+: no longer names the net of U5.21 (OUT2+), U6.2 (INL+)
- net OUTB-: no longer names the net of U5.22 (OUT2-), U6.1 (INL-)
- new net: C25.2, J4.24 (Pin_24)
- new net: C27.2, D4.1 (K), D5.2 (A)
- new net: Q2.1 (G), R7.1
- new net: C18.2, J4.5 (Pin_5)
- new net: C20.2, J4.18 (Pin_18)
- new net: C21.2, J4.20 (Pin_20)
- new net: C23.2, J4.22 (Pin_22)
- new net 3v3 OUT: C19.2, J4.15 (Pin_15), J4.16 (Pin_16)
- new net VGH: C22.2, D3.1 (K), J4.21 (Pin_21)
- new net VGL: C24.2, D4.2 (A), J4.23 (Pin_23)
- no-connect marks 7 -> 9
Other:
- note removed: "Audio"
- moved on the sheet: BT1, C1, C10, C11, C12, C13, C14, C15, C16, C17, C2, C4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

Commit message: Journal and sd cardgit add .
Parts:
- removed D1, D2: D_Small, symbol Device:D_Small
- added C29, C3: 1uF/50V, symbol Device:C_Small
- added D1: MBR0540, Diode_SMD:D_SOD-123, symbol Diode:MBR0540
- added J3: Micro_SD_Card, symbol Connector:Micro_SD_Card
- added Q1: DMG3414U, Package_TO_SOT_SMD:SOT-23, symbol Transistor_FET:DMG3414U
- added R10, R11, R12, R13, R14, R4: 10k, symbol Device:R_Small
- added R3: 100k, symbol Device:R_Small
Connections:
- net +3V3: now also J3.4 (VDD), R10.2, R11.2, R12.2, R13.2, R14.2, R4.2
- net +BATT: now also Q1.2 (S)
- net GND: now also C29.1, C3.1, J3.6 (VSS), J3.9 (SHIELD), R3.1
- net VBUS: now also C2.1, U3.3 (VI), D1.1 (K), D1.2 (A), Q1.1 (G), Q1.3 (D), R3.2
- net at J4.19 (Pin_19): now also C29.2
- net at J4.4 (Pin_4): now also C3.2
- net CLK: now reaches U1.11 (IO7)
- net CLK: now also J3.5 (CLK), R11.1
- net CMD: now reaches U1.12 (IO8)
- net CMD: now also J3.3 (CMD), R14.1
- net DAT0: now reaches U1.13 (IO9)
- net DAT0: now also J3.7 (DAT0), R12.1
- net DAT1: now reaches U1.25 (IO21)
- net DAT1: now also J3.8 (DAT1), R13.1
- net DAT2: now reaches U1.26 (IO26)
- net DAT2: now also J3.1 (DAT2), R4.1
- net DAT3: now reaches U1.35 (IO39)
- net DAT3: now also J3.2 (DAT3/CD), R10.1
- no-connect marks 9 -> 7
Other:
- moved on the sheet: BT1, C1, C10, C11, C12, C13, C14, C15, C16, C17, C2, C4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

Commit message: fix component issues
Connections:
- net +3V3: now also C15.1; no longer C15.2
- net GND: now also C14.2, C15.2; no longer C14.1, C15.1
- net at U6.12 (HPVDD): now also C14.1; no longer C14.2
Other:
- moved on the sheet: BT1, C18, C19, C20, C21, C22, C23, C24, C25, C26, C27, C28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

Commit message: NEW JOURNAL WOOP WOOP
Parts:
- removed J1: AudioJack3, symbol Connector_Audio:AudioJack3
- removed J3: Micro_SD_Card, symbol Connector:Micro_SD_Card
- removed Q1: DMG3414U, Package_TO_SOT_SMD:SOT-23, symbol Transistor_FET:DMG3414U
- added C30, C31: 4.7nF, Capacitor_SMD:C_0603_1608Metric_Pad1.08x0.95mm_HandSolder, symbol Device:C_Small
- added FB1: 600 Ω @ 100 MHz, footprints:FB_0603, symbol Device:FerriteBead_Small
- added J1: Micro_SD_Card_Det_Hirose_DM3AT, Connector_Card:microSD_HC_Hirose_DM3AT-SF-PEJM5, symbol Connector:Micro_SD_Card_Det_Hirose_DM3AT
- added J5: AudioJack3, footprints:SHOU-HAN-PJ-242, symbol Connector_Audio:AudioJack3_Ground_SwitchTR
- added Q3: AO3401A, Package_TO_SOT_SMD:SOT-23, symbol Transistor_FET:AO3401A
- added R15, R16, R17, R18: 1k, Resistor_SMD:R_0603_1608Metric, symbol Device:R_Small
- BT1: footprint (none) -> Connector_PinHeader_2.54mm:PinHeader_1x02_P2.54mm_Vertical
- C1, C10, C11, C12, C13, C14, C15, C16, C17, C18, C19, C2, C20, C21, C22, C23, C24, C25, C26, C27, C28, C29, C3, C4, C6, C8, C9: footprint (none) -> Capacitor_SMD:C_0603_1608Metric_Pad1.08x0.95mm_HandSolder
- C5, C7: value 1uF -> 0.1uF; footprint (none) -> Capacitor_SMD:C_0603_1608Metric_Pad1.08x0.95mm_HandSolder
- J2: footprint (none) -> Connector_USB:USB_C_Receptacle_HCTL_HC-TYPE-C-16P-01A
- J4: footprint (none) -> Connector_FFC-FPC:Amphenol_F32R-1A7x1-11024_1x24-1MP_P0.5mm_Horizontal
- L1: footprint (none) -> Inductor_SMD:L_0603_1608Metric
- R1, R10, R11, R12, R13, R14, R2, R3, R4, R5, R6, R7, R8, R9: footprint (none) -> Resistor_SMD:R_0603_1608Metric
- U2: footprint leptosis:WLP-8_1.67x0.93_P0.4 -> smth:WLP-8_1.67x0.93_P0.4
- U5: footprint Library:Texas_RGE0024R_VQFN-24-1EP_4x4mm_P0.5mm_EP2.1x2.1mm -> footprints:Texas_RGE0024R_VQFN-24-1EP_4x4mm_P0.5mm_EP2.1x2.1mm
Connections:
- net +3.3VA: now also FB1.2
- net +3V3: now also FB1.1, J1.4 (VDD)
- net +BATT: now also Q3.3 (D)
- net CLK: now also J1.5 (CLK)
- net CMD: now also J1.3 (CMD)
- net DAT0: now also J1.7 (DAT0)
- net DAT1: now also J1.8 (DAT1)
- net DAT2: now also J1.1 (DAT2)
- net DAT3: now also J1.2 (DAT3/CD)
- net EN: now also U1.27 (IO47)
- net G0: now also U1.41 (IO45)
- net G1: now also U1.44 (IO46)
- net GND: now also SW7.1, J1.11 (SHIELD), J1.6 (VSS), J1.9 (DET_B), J5.G, J5.S; no longer SW7.2
- net VBUS: now also Q3.1 (G), Q3.2 (S)
- net at U5.19 (OUT1-): now also R16.1; no longer U6.4 (INR-)
- net at U6.3 (INR+): now also C30.1, R15.2; no longer U5.20 (OUT1+)
- net at U6.2 (INL+): now also C31.1, R17.2; no longer U5.21 (OUT2+)
- net at U6.1 (INL-): now also C31.2, R18.2; no longer U5.22 (OUT2-)
- net DET_A: now reaches U1.7 (IO3)
- net DET_A: now also J1.10 (DET_A)
- net LEFT: no longer names the net of U6.16 (OUTL)
- net LEFT: now also J5.T
- net RIGHT: no longer names the net of U6.5 (OUTR)
- net RIGHT: now also J5.R
- net ~{RESET}: no longer names the net of C28.2, R9.1, U1.45 (EN)
- net ~{RESET}: now also SW7.2; no longer SW7.1
- new net: C30.2, R16.2, U6.4 (INR-)
- new net: R15.1, U5.20 (OUT1+)
- new net: R17.1, U5.21 (OUT2+)
- new net: R18.1, U5.22 (OUT2-)
- no-connect marks 7 -> 9
Other:
- moved on the sheet: C10, C11, C12, C13, C14, C15, C16, C17, C18, C19, C20, C21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

Commit message: new thingies and new file
Parts:
- added C32: 1uF, Capacitor_SMD:C_0603_1608Metric_Pad1.08x0.95mm_HandSolder, symbol Device:C_Small
- added C33: 10uF, Capacitor_SMD:C_0603_1608Metric_Pad1.08x0.95mm_HandSolder, symbol Device:C_Small
- added C34: 0.1uF, Capacitor_SMD:C_0603_1608Metric_Pad1.08x0.95mm_HandSolder, symbol Device:C_Small
- added D2: 1N4148W, Diode_SMD:D_SOD-123, symbol Diode:1N4148W
- added Q1: PMOS, symbol Simulation_SPICE:PMOS
- added Q4: NMOS, symbol Simulation_SPICE:NMOS
- added R19: 10k, symbol Device:R_Small
- added R20, R22: 100k, symbol Device:R_Small
- added R21: 300k, symbol Device:R_Small
Connections:
- net +BATT: now also Q1.3 (S), R19.1, R20.1; no longer Q3.3 (D)
- net GND: now also SW1.1, C34.1, Q4.3 (S); no longer SW1.2
- net SW_1: no longer names the net of U1.17 (IO13)
- net SW_1: no longer SW1.1
- new net: C32.1, D2.1 (K), R19.2, SW1.2
- new net: C32.2, C34.2, Q1.2 (G), Q4.1 (D), R20.2
- new net: C33.1, Q4.2 (G), R21.1
- new net: D2.2 (A), R21.2, R22.2
- new net BAT_OUT: C33.2, Q1.1 (D), Q3.3 (D), R22.1
- no-connect marks 9 -> 10
Other:
- moved on the sheet: C10, C11, C12, C13, C14, C15, C18, C19, C20, C21, C22, C23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
